File: Power Distribution Senior/MCU.kicad_sch (KiCad schematic)
At the start: 19 parts, among them J4 Conn_01x04_Pin, SW1 SW_SPDT, U7 STM32G474RETx, X1 X322516MLB4SI

Commit message: Added FootPrints
Parts:
- removed C41, C42: 8pF, symbol Device:C_Small
- removed X1: X322516MLB4SI, easyeda2kicad:OSC-SMD_4P-L3.2-W2.5-BL, symbol YXC Crystal Oscillators X322516MLB4SI:X322516MLB4SI
- added C43: 10nF, Capacitor_SMD:C_0603_1608Metric, symbol Device:C_Small
- added OSC1: ASE-8.000MHZ-LC-T, ABRACON ASE-8.000MHZ-LC-T:OSC-SMD_4P-L3.2-W2.5-CJ13-320001210A20, symbol ABRACON ASE-8.000MHZ-LC-T:ASE-8.000MHZ-LC-T
- C17: value 10u -> 10uF; footprint Capacitor_SMD:C_0603_1608Metric -> Capacitor_SMD:C_1210_3225Metric
- C18, C19, C20, C21, C25: value 100n -> 0.1uF
- C22, C23, C24: footprint Capacitor_SMD:C_0402_1005Metric -> Capacitor_SMD:C_0603_1608Metric
- C39, C40: value 100nF -> 0.1uF; footprint (none) -> Capacitor_SMD:C_0603_1608Metric
- R34: footprint (none) -> Resistor_SMD:R_0402_1005Metric
Connections:
- net +3.3V: now also C43.1, OSC1.1 (Tri/STBY), OSC1.4 (VDD)
- net GND: now also C43.2, OSC1.2 (GND)
- net RCC_OSC_IN: now also OSC1.3 (OUT)
- net CHARGE_EN: now reaches U7.12 (PA0)
Other:
- note removed: "(9-5)*2=8"
- note removed: "9pF"

Commit message: Updated pcb
Parts:
- removed SW1: SW_SPDT, Button_Switch_SMD:SW_SPDT_PCM12, symbol Switch:SW_SPDT
- C17: footprint Capacitor_SMD:C_1210_3225Metric -> Capacitor_SMD:C_0805_2012Metric
Connections:
- net SW_BOOT0 is gone; now on net GND: R34.1
- net INA226_ALERT_1: now also U7.39 (PC7); no longer U7.2 (PC13)
- net INA226_ALERT_2: now also U7.44 (PA10); no longer U7.3 (PC14)
- net LORA_DIO0: now also U7.26 (PB2); no longer U7.25 (PB1)
- net LORA_DIO1: now also U7.25 (PB1); no longer U7.26 (PB2)
- net IMU2_INT1: now reaches U7.10 (PC2)
- net LORA_DIO2: now reaches U7.17 (PA3)
- net IMU2_SCLK: now reaches U7.52 (PC10)
- net IMU2_MISO: now reaches U7.53 (PC11)
- net IMU2_MOSI: now reaches U7.54 (PC12)
- net IMU1_INT1: now reaches U7.9 (PC1)
- net SPI2_CS renamed IMU1_CS
- net SPI2_MISO renamed IMU1_MISO
- net SPI2_MOSI renamed IMU1_MOSI
- net SPI2_SCK renamed IMU1_SCLK
- new net IMU2_CS: U7.2 (PC13)
- no-connect marks 2 -> 18
Other:
- note added: "Pull down to gnd"
- note added: "Reaction wheel Primary IMU"
- note added: "Reaction wheel Secondary IMU"
- note removed: "Toggle the button. Program Toggle back."
