File: Power Distribution Senior/Power Distribution Senior.kicad_sch (KiCad schematic)
At the start: 92 parts, among them J1 Conn_Coaxial, J2 Conn_01x02_Socket, J3 Conn_01x02_Socket, Q1 SI7288DP-T1-GE3, Q2 SI7288DP-T1-GE3, Q3 2N7002, Q4 AO3401A, Q5 AO3407A, U1 BQ24650, U2 AP63205WU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

Commit message: Added FootPrints
Parts:
- removed J2, J3: Conn_01x02_Socket, TerminalBlock:TerminalBlock_bornier-2_P5.08mm, symbol Connector:Screw_Terminal_01x02
- added SW3: SW_SPST, symbol Switch:SW_SPST
- added TP1: + Solar, TestPoint:TestPoint_Pad_4.0x4.0mm, symbol Connector:TestPoint
- added TP2: - Solar, TestPoint:TestPoint_Pad_4.0x4.0mm, symbol Connector:TestPoint
- added TP3, TP4: 5V Motor, TestPoint:TestPoint_Pad_3.0x3.0mm, symbol Connector:TestPoint
- added TP5, TP6: 3.3V, TestPoint:TestPoint_Pad_3.0x3.0mm, symbol Connector:TestPoint
- added TP7: + Battery, TestPoint:TestPoint_Pad_4.0x4.0mm, symbol Connector:TestPoint
- added TP8: - Battery, TestPoint:TestPoint_Pad_4.0x4.0mm, symbol Connector:TestPoint
- C1, C11, C27, C30, C31, C34, C4, C6, C8: footprint (none) -> Capacitor_SMD:C_1210_3225Metric
- C10, C12, C13, C14, C15, C16, C2, C3, C35, C36, C5, C7: footprint (none) -> Capacitor_SMD:C_0805_2012Metric
- C26, C28, C29, C32, C37, C38: footprint (none) -> Capacitor_SMD:C_0603_1608Metric
- C33: value 100nF -> 0.1uF; footprint (none) -> Capacitor_SMD:C_0603_1608Metric
- C9: footprint (none) -> Capacitor_SMD:C_0201_0603Metric
- D1, D8, D9: footprint (none) -> LED_SMD:LED_0603_1608Metric
- R1, R19, R20, R21, R22, R28, R29, R30, R31, R32, R33, R35, R36: footprint (none) -> Resistor_SMD:R_0805_2012Metric
- R10, R11, R12, R13, R14, R15, R17, R18, R2, R26, R27, R3, R4, R5, R6, R7, R8: footprint (none) -> Resistor_SMD:R_0402_1005Metric
- R16, R23: footprint (none) -> Resistor_SMD:R_2512_6332Metric
- R24, R25: footprint (none) -> Resistor_SMD:R_0603_1608Metric
- R9: footprint (none) -> Resistor_SMD:R_1206_3216Metric
- RSR1: footprint Resistor_SMD:R_1206_3216Metric -> Resistor_SMD:R_2512_6332Metric
- U5: footprint easyeda2kicad:SMD-22_L37.0-W25.0-P2.54-LB -> DreamLNK DL-SX1278PA:SMD-22_L37.0-W25.0-P2.54-LB
- U8: footprint easyeda2kicad:LL-34_L3.5-W1.5-RD -> HXY MOSFET ZMM15V:LL-34_L3.5-W1.5-RD
Connections:
- net +3.3V: now also TP5.1, TP6.1
- net +5V: now also TP3.1, TP4.1
- net BAT_CHARGE: now also SW3.1 (A)
- net GND: now also TP2.1, TP8.1
- net V_SOLAR: now also TP1.1
- new net: SW3.2 (B), TP7.1
Other:
- note removed: "+"
- note removed: "-"

Commit message: Updated pcb
Parts:
- removed C11, C27, C30, C31: 10uF, Capacitor_SMD:C_1210_3225Metric, symbol Device:C_Small
- removed C12: 0.1uF, Capacitor_SMD:C_0805_2012Metric, symbol Device:C_Small
- removed C13, C14: 22uF, Capacitor_SMD:C_0805_2012Metric, symbol Device:C_Small
- removed C15: 1uF, Capacitor_SMD:C_0805_2012Metric, symbol Device:C_Small
- removed C16: 1000pF, Capacitor_SMD:C_0805_2012Metric, symbol Device:C_Small
- removed C26, C28, C29, C32, C37, C38: 0.1uF, Capacitor_SMD:C_0603_1608Metric, symbol Device:C_Small
- removed D1, D8: LED, LED_SMD:LED_0603_1608Metric, symbol Device:LED
- removed D6: PTVS26VZ1USK, Diode_SMD:Nexperia_DSN1608-2_1.6x0.8mm, symbol Diode:PTVS26VZ1USK
- removed D7: PTVS10VZ1USK, Diode_SMD:Nexperia_DSN1608-2_1.6x0.8mm, symbol Diode:PTVS10VZ1USK
- removed L2: 4.7uH, Inductor_SMD:L_Vishay_IFSC-1515AH_4x4x1.8mm, symbol Device:L
- removed Q4: AO3401A, AO3401A:SOT23-3, symbol AO3401A:AO3401A
- removed Q5: AO3407A, AO3407A:SOT95P280X125-3N, symbol AO3407A:AO3407A
- removed R11: 332k, Resistor_SMD:R_0402_1005Metric, symbol Device:R_Small
- removed R12: 47k, Resistor_SMD:R_0402_1005Metric, symbol Device:R_Small
- removed R13, R15: 8.2, Resistor_SMD:R_0402_1005Metric, symbol Device:R_Small
- removed R14: 330, Resistor_SMD:R_0402_1005Metric, symbol Device:R_Small
- removed R16, R23: 20m, Resistor_SMD:R_2512_6332Metric, symbol Device:R_Small
- removed R17, R18, R26, R27: 10k, Resistor_SMD:R_0402_1005Metric, symbol Device:R_Small
- removed R19, R20, R21, R22, R28, R29, R31: 0, Resistor_SMD:R_0805_2012Metric, symbol Device:R_Small
- removed R24, R25: 10, Resistor_SMD:R_0603_1608Metric, symbol Device:R_Small
- removed R30, R33: 100k, Resistor_SMD:R_0805_2012Metric, symbol Device:R_Small
- removed R35: 1k, Resistor_SMD:R_0805_2012Metric, symbol Device:R_Small
- removed SW3: SW_SPST, symbol Switch:SW_SPST
- removed U2: AP63205WU, Package_TO_SOT_SMD:TSOT-23-6, symbol Regulator_Switching:AP63205WU
- removed U3, U4: INA226, Package_SO:VSSOP-10_3x3mm_P0.5mm, symbol Sensor_Energy:INA226
- removed U6: MCP1727-ADJxMF, Package_DFN_QFN:DFN-8-1EP_3x3mm_P0.65mm_EP1.55x2.4mm, symbol Regulator_Linear:MCP1727-ADJxMF
- removed U8: ZMM15V, HXY MOSFET ZMM15V:LL-34_L3.5-W1.5-RD, symbol HXY MOSFET ZMM15V:ZMM15V_C5346000
- added H1, H2, H3, H4: MountingHole, MountingHole:MountingHole_3.2mm_M3_DIN965_Pad, symbol Mechanical:MountingHole
- C1, C34, C8: footprint Capacitor_SMD:C_1210_3225Metric -> Capacitor_SMD:C_1206_3216Metric
- C35, C36: footprint Capacitor_SMD:C_0805_2012Metric -> Capacitor_SMD:C_0603_1608Metric
- C4, C6: footprint Capacitor_SMD:C_1210_3225Metric -> Capacitor_SMD:C_0805_2012Metric
- C9: footprint Capacitor_SMD:C_0201_0603Metric -> Capacitor_SMD:C_0402_1005Metric
- J1: footprint (none) -> HRS U.FL-R-SMT-1(80):RF-SMD_FRF05002-JSS103M
- TP5, TP6: value 3.3V -> GND
Connections:
- net +3.3V is gone; now on net GND: TP5.1, TP6.1
- net BAT_CHARGE is gone; now on net VBAT_RAW: C6.1, C7.1, C8.1, C9.1, R2.1, RSR1.2, U1.9 (SRN)
- net +5V: no longer TP3.1, TP4.1
- net GND: now also U1.17 (GND)
- net VBAT_PROTECTED: now also TP3.1, TP4.1
- net VBAT_RAW: now also TP7.1
- net V_SOLAR_MEASURED: now reaches C4.1, D4.3, Q1.5_6_10, R9.1
- net DIO0 renamed LORA_DIO0
- net DIO1 renamed LORA_DIO1
- net DIO2 renamed LORA_DIO2
Other:
- added sheet IMU (IMU.kicad_sch)
- added sheet Monitoring (Monitoring.kicad_sch)
- added sheet Protection (Protection.kicad_sch)
- added sheet Regulators (Regulators.kicad_sch)
- note added: "3C 3000mAh from edison"
- note added: "Either remove the switch or find a good spst switch"
- note added: "Mounting Holes"
- note added: "this is a current output from bq24650. it doesnt need to have a seperate pwr flag and output"
- note removed: "1.5A LDO Takes 2.3-6V"
- note removed: "20VGS"
- note removed: "3.3V Rail"
- note removed: "5V Rail"
- note removed: "5V Regulator"
- note removed: "Battery -> Power Rails"
- note removed: "Battery Connection"
- note removed: "Battery Protection"
- note removed: "Change values to match battery voltage not solar"
- note removed: "Charging Logic"
- note removed: "Connect Solar charger directly to battery. then before the connection to the rails add a filter."
- note removed: "Done using bq24650 inbuilt logic"
- note removed: "Filtering"
- note removed: "LED = ON , stable and good to use"
- note removed: "Power Monitoring"
- note removed: "Reverse bias diode?"
- note removed: "Solar Protection"
- note removed: "Solar panel -> Solar charge controller"
- note removed: "Using equation from datasheet to get the values of R2 and R1"
- note removed: "VBAT+"
- note removed: "VS takes 5v from battery to power it up"
- note removed: "should connect to vbus of 5V RAIL"
- note removed: "should connect to vbus of mppt"
- note removed: "this is grounded from the mppt"
- note removed: "tvs diode for protection of spikes"
- note removed: "zener diode instead of clamping it regulates the voltage in vgs to be constantly around 15v"
- note removed: "zener diode prevents vgs from reaching more than 20, clamps at 15v"
- moved on the sheet: C33, C34, C35, C36, J1, R32, TP3, TP4, TP5, TP6, TP7, TP8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
